File: kicad/utcs-isource.kicad_pcb (KiCad board)
At the start: 2 copper layers, 101.6 x 101.6 mm, 34 parts, among them J1 Conn_01x06, J2 Conn_01x03, P1 CONN_2, U1 AD5660, U2 AD8221, U3 OP1177

Commit message: Initial P1 Fab
Routing:
- net (no net): vias 0 -> 6
- added copper zone on F.Cu, net GND
Changed lines of the file:
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@@
   (general
     (links 63)
-    (no_connects 24)
-    (area 50.724999 25.324999 152.475001 127.075001)
+    (no_connects 3)
+    (area 25.324999 -150.044 150.473138 128.891)
     (thickness 1.6)
     (drawings 8)
-    (tracks 154)
+    (tracks 160)
     (zones 0)
     (modules 34)
@@
     (via_min_size 0.381)
     (via_min_drill 0.254)
-    (user_via 1.778 1.0922)
+    (user_via 2.54 1.016)
     (uvia_size 0.2794)
     (uvia_drill 0.1016)
@@
       (net 2 GND))
   )
-  (gr_text "utcs-isource (prototype single-channel)\nProgrammable 0.1-100uA Current Source\n\nCopyright 2017\nDesigned By: Andrey K. Shmakov\ngithub.com/akshmakov/utcs-isource" (at 102.616 35.052) (layer F.SilkS)
+  (gr_text "utcs-isource (prototype single-channel)\nProgrammable 0.1-100uA Current Source\n\nCopyright 2017\nDesigned By: Andrey K. Shmakov\ngithub.com/akshmakov/utcs-isource" (at 45.72 121.92 90) (layer F.SilkS)
     (effects (font (size 1.5 1.5) (thickness 0.3)) (justify left))
   )
-  (gr_text "SN:\n" (at 96.52 111.125) (layer F.SilkS)
+  (gr_text "SN:\n" (at 83.312 114.808) (layer F.SilkS)
     (effects (font (size 1.5 1.5) (thickness 0.3)))
   )
-  (gr_text "PCA P/N :  UTCS-ISOURCE-ASSY-1 \n\n               - REV:" (at 94.615 99.695) (layer F.SilkS)
+  (gr_text "PCA P/N :  UTCS-ISOURCE-ASSY-1 \n\n               - REV:" (at 82.804 88.9) (layer F.SilkS)
     (effects (font (size 1.5 1.5) (thickness 0.3)) (justify left))
   )
-  (gr_text "PCB P/N :  UTCS-ISOURCE-1 \n\n               - REV:\n" (at 94.615 89.535) (layer F.SilkS)
+  (gr_text "PCB P/N :  UTCS-ISOURCE-1 \n\n               - REV:\n" (at 83.312 78.232) (layer F.SilkS)
     (effects (font (size 1.5 1.5) (thickness 0.3)) (justify left))
   )
-  (gr_line (start 50.8 25.4) (end 50.8 127) (angle 90) (layer Edge.Cuts) (width 0.15))
-  (gr_line (start 152.4 25.4) (end 50.8 25.4) (angle 90) (layer Edge.Cuts) (width 0.15))
-  (gr_line (start 152.4 127) (end 152.4 25.4) (angle 90) (layer Edge.Cuts) (width 0.15))
-  (gr_line (start 50.8 127) (end 152.4 127) (angle 90) (layer Edge.Cuts) (width 0.15))
+  (gr_line (start 25.4 25.4) (end 25.4 127) (angle 90) (layer Edge.Cuts) (width 0.15))
+  (gr_line (start 127 25.4) (end 25.4 25.4) (angle 90) (layer Edge.Cuts) (width 0.15))
+  (gr_line (start 127 127) (end 127 25.4) (angle 90) (layer Edge.Cuts) (width 0.15))
+  (gr_line (start 25.4 127) (end 127 127) (angle 90) (layer Edge.Cuts) (width 0.15))
+  (via (at 121.92 121.92) (size 2.54) (drill 1.016) (layers F.Cu B.Cu) (net 0))
+  (via (at 30.48 121.92) (size 2.54) (drill 1.016) (layers F.Cu B.Cu) (net 0))
+  (via (at 30.48 30.48) (size 2.54) (drill 1.016) (layers F.Cu B.Cu) (net 0))
+  (via (at 121.92 30.48) (size 2.54) (drill 1.016) (layers F.Cu B.Cu) (net 0))
+  (via (at 30.48 76.2) (size 2.54) (drill 1.016) (layers F.Cu B.Cu) (net 0))
+  (via (at 121.92 76.2) (size 2.54) (drill 1.016) (layers F.Cu B.Cu) (net 0))
   (segment (start 74.95 88.265) (end 74.93 88.265) (width 0.3556) (layer F.Cu) (net 1))
   (segment (start 74.93 88.265) (end 73.66 89.535) (width 0.3556) (layer F.Cu) (net 1))
@@
     (connect_pads yes (clearance 0.635))
     (min_thickness 0.254)
-    (fill (arc_segments 16) (thermal_gap 0.508) (thermal_bridge_width 0.508))
+    (fill yes (arc_segments 16) (thermal_gap 0.508) (thermal_bridge_width 0.508))
     (polygon
       (pts
         (xy 64.135 70.485) (xy 60.325 66.675) (xy 60.325 57.15) (xy 59.055 55.88) (xy 59.055 25.4)
-        (xy 152.4 25.4) (xy 152.4 127) (xy 50.8 127) (xy 50.8 77.47) (xy 64.135 77.47)
+        (xy 127 25.4) (xy 127 127) (xy 25.4 127) (xy 25.4 77.47) (xy 64.135 77.47)
       )
     )
@@
     (connect_pads yes (clearance 0.635))
     (min_thickness 0.254)
-    (fill (arc_segments 16) (thermal_gap 0.508) (thermal_bridge_width 0.508))
+    (fill yes (arc_segments 16) (thermal_gap 0.508) (thermal_bridge_width 0.508))
     (polygon
       (pts
         (xy 54.61 76.835) (xy 63.5 76.835) (xy 63.5 71.12) (xy 59.055 66.675) (xy 59.055 57.15)
-        (xy 57.785 55.88) (xy 57.785 25.4) (xy 50.8 25.4) (xy 50.8 76.835) (xy 55.245 76.835)
+        (xy 57.785 55.88) (xy 57.785 25.4) (xy 25.4 25.4) (xy 25.4 76.835) (xy 55.245 76.835)
       )
     )
@@
     (connect_pads yes (clearance 0.635))
     (min_thickness 0.254)
-    (fill (arc_segments 16) (thermal_gap 0.508) (thermal_bridge_width 0.508))
+    (fill yes (arc_segments 16) (thermal_gap 0.508) (thermal_bridge_width 0.508))
     (polygon
       (pts
@@
     (polygon
       (pts
-        (xy 127.254 94.742) (xy 120.904 94.742) (xy 120.904 89.662) (xy 127.254 89.662)
+        (xy 116.078 83.566) (xy 109.728 83.566) (xy 109.728 78.486) (xy 116.078 78.486)
       )
     )
@@
     (polygon
       (pts
-        (xy 127.254 105.41) (xy 120.904 105.41) (xy 120.904 100.33) (xy 127.254 100.33)
+        (xy 116.586 94.234) (xy 110.236 94.234) (xy 110.236 89.154) (xy 116.586 89.154)
       )
     )
@@
     (polygon
       (pts
-        (xy 127.254 113.538) (xy 99.568 113.538) (xy 99.568 109.728) (xy 127.254 109.728)
+        (xy 114.554 117.094) (xy 86.868 117.094) (xy 86.868 113.284) (xy 114.554 113.284)
       )
     )
+  )
+  (zone (net 2) (net_name GND) (layer F.Cu) (hatch edge 0.508)
+    (connect_pads yes (clearance 0.635))
+    (min_thickness 0.254)
+    (fill yes (arc_segments 16) (thermal_gap 0.508) (thermal_bridge_width 0.508))
+    (polygon
+      (pts
+        (xy 62.992 52.324) (xy 58.928 56.388) (xy 58.928 66.548) (xy 64.516 72.136) (xy 66.04 72.136)
+        (xy 66.04 67.564) (xy 65.024 66.548) (xy 65.024 59.944) (xy 73.152 51.816) (xy 86.36 51.816)
+        (xy 91.44 56.896) (xy 97.536 56.896) (xy 97.536 25.4) (xy 127 25.4) (xy 127 127)
+        (xy 25.4 127) (xy 25.4 25.4) (xy 62.992 25.4)
+      )
+    )

Commit message: Updated to double sided plating for through hole components
Parts:
- added MNT1: TEST_1P, Mounting_Holes:MountingHole_4.5mm_Pad, F.Cu at (33.0, 33.0)
- added MNT2: TEST_1P, Mounting_Holes:MountingHole_4.5mm_Pad, F.Cu at (119.4, 33.0)
- added MNT3: TEST_1P, Mounting_Holes:MountingHole_4.5mm_Pad, F.Cu at (33.0, 76.2)
- added MNT4: TEST_1P, Mounting_Holes:MountingHole_4.5mm_Pad, F.Cu at (33.0, 119.4)
- added MNT5: TEST_1P, Mounting_Holes:MountingHole_4.5mm_Pad, F.Cu at (119.4, 119.4)
- added MNT6: TEST_1P, Mounting_Holes:MountingHole_4.5mm_Pad, F.Cu at (119.4, 76.2)
Routing:
- net (no net): vias 6 -> 0
